Commit message: Add base link

File: src/rai_description/robot.urdf (robot description, URDF)
Before this commit: robot robot, 10 links, 9 joints
Links:
- added link base_link, mass 0
Joints:
- added joint base_link_to_chassis: type fixed, parent base_link, child chassis, origin xyz=0 0 0 rpy=0 -0 0, axis 0 0 1, limit effort=10 velocity=10

Commit message: Change assets to meshes to match industry standard

File: src/rai_description/robot.urdf (robot description, URDF)
Before this commit: robot robot, 11 links, 10 joints
Links:
- link arm: geometry collision box size=0.51 0.03 0.03; collision cylinder length=0.06 radius=0.025
- link arm_2: geometry collision box size=0.51 0.03 0.03; collision cylinder length=0.06 radius=0.025
- link arm_3: geometry collision box size=0.51 0.03 0.03; collision cylinder length=0.06 radius=0.025
- link arm_4: geometry collision box size=0.51 0.03 0.03; collision cylinder length=0.06 radius=0.025
- link arm_gantry: geometry visual mesh filename=package://rai_description/meshes/merged/arm_gantry_visual.s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
- link arm_gantry_2: geometry visual mesh filename=package://rai_description/meshes/merged/arm_gantry_2_visual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
- link arm_gantry_3: geometry visual mesh filename=package://rai_description/meshes/merged/arm_gantry_3_visual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
- link arm_gantry_4: geometry visual mesh filename=package://rai_description/meshes/merged/arm_gantry_4_visual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
- link canvas: geometry visual mesh filename=package://rai_description/meshes/merged/canvas_visual.stl
- link chassis: geometry visual mesh filename=package://rai_description/meshes/merged/chassis_visual.stl
