Commit message: add sim enabled env

File: src/rai_description/urdf/rai.urdf.xacro (robot description, xacro)
@@ -3,3 +3,8 @@
     <!-- Include generated urdf -->
     <xacro:include filename="$(find rai_description)/urdf/rai_geometry.urdf" />
+    <link name="world"/>
+    <joint name="world_fixed" type="fixed">
+        <parent link="world"/>
+        <child link="base_link"/>
+    </joint>
 </robot>
