Commit message: placeholder implementations

File: src/rai_description/urdf/rai.ros2_control.xacro (robot description, xacro)
@@ -1,5 +1,17 @@
 <?xml version="1.0"?>
 <robot xmlns:xacro="http://www.ros.org/wiki/xacro">
-  <xacro:macro name="bot_ros2_control" params="name prefix use_mock_hardware">
+  <xacro:macro name="arm_revolute_macro" params="prefix id use_mock_hardware">
+    <ros2_control name="${prefix}_${name}_HW" type="system">
+      <hardware>
+        <plugin>ros2_control_demo_hardware/MySystemHardware</plugin>
+      </hardware>
+      <joint name="${prefix}_${name}_joint">
+        <command_interface name="position"/>
+        <state_interface name="position"/>
+        <state_interface name="velocity"/>
+      </joint>
+    </ros2_control>
+  </xacro:macro>
+  <xacro:macro name="rai_ros2_control" params="name prefix use_mock_hardware">
     <ros2_control name="${name}" type="system">
       <!-- Physical hardware plugin-->

File: src/rai_description/urdf/rai.urdf.xacro (robot description, xacro)
@@ -1,4 +1,6 @@
 <?xml version="1.0"?>
 <robot name="rai" xmlns:xacro="http://www.ros.org/wiki/xacro">
+    <xacro:arg name="use_sim" default="false"/>
+    <xacro:arg name="use_mock_hardware" default="false"/>
     <!-- Include generated urdf -->
     <xacro:include filename="$(find rai_description)/urdf/rai_geometry.urdf" />

Commit message: intermediate commit, before changing mock hardware params to args

File: src/rai_description/urdf/rai.ros2_control.xacro (robot description, xacro)
@@ -1,10 +1,27 @@
 <?xml version="1.0"?>
 <robot xmlns:xacro="http://www.ros.org/wiki/xacro">
-  <xacro:macro name="arm_revolute_macro" params="prefix id use_mock_hardware">
-    <ros2_control name="${prefix}_${name}_HW" type="system">
-      <hardware>
-        <plugin>ros2_control_demo_hardware/MySystemHardware</plugin>
-      </hardware>
-      <joint name="${prefix}_${name}_joint">
+  <xacro:macro name="arm_macro" params="id use_sim use_mock_hardware">
+    <ros2_control name="arm_${id}" type="system">
+      <xacro:unless value="${use_mock_hardware}">
+        <hardware>
+          <plugin></plugin> #TODO Placeholder for real hardware
+        </hardware>
+      </xacro:unless>
+      <xacro:if value="${use_mock_hardware and use_sim}">
+        <hardware>
+          <plugin>gz_ros2_control/GazeboSimSystem</plugin>
+        </hardware>
+      </xacro:unless>
+      <xacro:if value="${use_mock_hardware and not use_sim}">
+        <hardware>
+          <plugin>mock_components/GenericSystem</plugin>
+        </hardware>
+      </xacro:unless>
+      <joint name="$arm_revolute_${id}">
+        <command_interface name="position"/>
+        <state_interface name="position"/>
+        <state_interface name="velocity"/>
+      </joint>
+      <joint name="$arm_slider_${id}">
         <command_interface name="position"/>
         <state_interface name="position"/>
@@ -13,34 +30,30 @@
     </ros2_control>
   </xacro:macro>
-  <xacro:macro name="rai_ros2_control" params="name prefix use_mock_hardware">
-    <ros2_control name="${name}" type="system">
-      <!-- Physical hardware plugin-->
+  <ros2_control name="canvas" type="system">
       <xacro:unless value="${use_mock_hardware}">
         <hardware>
-          <plugin>odrive_ros2_control_plugin/ODriveHardwareInterface</plugin>
-          <param name="can">can0</param>
+          <plugin></plugin> #TODO Placeholder for real hardware
         </hardware>
       </xacro:unless>
-      <!-- Generic mock hardware motors-->
-      <!-- TODO Make it so that GazeboSimSystem is dependent on use_sim, and GenericSystem is dependent on !use_sim and use_mock_hardware-->
-      <xacro:if value="${use_mock_hardware}">
+      <xacro:if value="${use_mock_hardware and use_sim}">
         <hardware>
           <plugin>gz_ros2_control/GazeboSimSystem</plugin>
         </hardware>
-      </xacro:if>
-      <!-- Odrive node ID setups-->
-      <joint name="${prefix}left_wheel_joint">
-        <param name="node_id">0</param>
-         <command_interface name="velocity"/>
+      </xacro:unless>
+      <xacro:if value="${use_mock_hardware and not use_sim}">
+        <hardware>
+          <plugin>mock_components/GenericSystem</plugin>
+        </hardware>
+      </xacro:unless>
+      <joint name="$arm_revolute_${id}">
+        <command_interface name="position"/>
         <state_interface name="position"/>
         <state_interface name="velocity"/>
       </joint>
-      <joint name="${prefix}right_wheel_joint">
-        <param name="node_id">1</param>
-         <command_interface name="velocity"/>
+      <joint name="$arm_slider_${id}">
+        <command_interface name="position"/>
         <state_interface name="position"/>
         <state_interface name="velocity"/>
       </joint>
     </ros2_control>
-  </xacro:macro>
 </robot>

File: src/rai_description/urdf/rai.urdf.xacro (robot description, xacro)
@@ -5,4 +5,5 @@
     <!-- Include generated urdf -->
     <xacro:include filename="$(find rai_description)/urdf/rai_geometry.urdf" />
+    <xacro:include filename="$(find igvc_description)/control/bot.ros2_control.xacro" />
     <link name="world"/>
     <joint name="world_fixed" type="fixed">
@@ -10,3 +11,7 @@
         <child link="base_link"/>
     </joint>
+    <xacro:arm_macro id ="1"/>
+    <xacro:arm_macro id ="2"/>
+    <xacro:arm_macro id ="3"/>
+    <xacro:arm_macro id ="4"/>
 </robot>

Commit message: change params to args, add canvas

File: src/rai_description/urdf/rai.ros2_control.xacro (robot description, xacro)
@@ -3,15 +3,15 @@
   <xacro:macro name="arm_macro" params="id use_sim use_mock_hardware">
     <ros2_control name="arm_${id}" type="system">
-      <xacro:unless value="${use_mock_hardware}">
+      <xacro:unless value="$(arg use_mock_hardware)">
         <hardware>
           <plugin></plugin> #TODO Placeholder for real hardware
         </hardware>
       </xacro:unless>
-      <xacro:if value="${use_mock_hardware and use_sim}">
+      <xacro:if value="${$(arg use_mock_hardware) and $(arg use_sim)}">
         <hardware>
           <plugin>gz_ros2_control/GazeboSimSystem</plugin>
         </hardware>
       </xacro:unless>
-      <xacro:if value="${use_mock_hardware and not use_sim}">
+      <xacro:if value="${$(arg use_mock_hardware) and not $(arg use_sim)}">
         <hardware>
           <plugin>mock_components/GenericSystem</plugin>
@@ -31,29 +31,24 @@
   </xacro:macro>
   <ros2_control name="canvas" type="system">
-      <xacro:unless value="${use_mock_hardware}">
-        <hardware>
-          <plugin></plugin> #TODO Placeholder for real hardware
-        </hardware>
-      </xacro:unless>
-      <xacro:if value="${use_mock_hardware and use_sim}">
-        <hardware>
-          <plugin>gz_ros2_control/GazeboSimSystem</plugin>
-        </hardware>
-      </xacro:unless>
-      <xacro:if value="${use_mock_hardware and not use_sim}">
-        <hardware>
-          <plugin>mock_components/GenericSystem</plugin>
-        </hardware>
-      </xacro:unless>
-      <joint name="$arm_revolute_${id}">
-        <command_interface name="position"/>
-        <state_interface name="position"/>
-        <state_interface name="velocity"/>
-      </joint>
-      <joint name="$arm_slider_${id}">
-        <command_interface name="position"/>
-        <state_interface name="position"/>
-        <state_interface name="velocity"/>
-      </joint>
-    </ros2_control>
+    <xacro:unless value="$(arg use_mock_hardware)">
+      <hardware>
+        <plugin></plugin> #TODO Placeholder for real hardware
+      </hardware>
+    </xacro:unless>
+    <xacro:if value="${$(arg use_mock_hardware) and $(arg use_sim)}">
+      <hardware>
+        <plugin>gz_ros2_control/GazeboSimSystem</plugin>
+      </hardware>
+    </xacro:unless>
+    <xacro:if value="${$(arg use_mock_hardware) and not $(arg use_sim)}">
+      <hardware>
+        <plugin>mock_components/GenericSystem</plugin>
+      </hardware>
+    </xacro:unless>
+    <joint name="$canvas_revolute">
+      <command_interface name="position"/>
+      <state_interface name="position"/>
+      <state_interface name="velocity"/>
+    </joint>
+  </ros2_control>
 </robot>

Commit message: remove params from arm macro

File: src/rai_description/urdf/rai.ros2_control.xacro (robot description, xacro)
@@ -1,5 +1,5 @@
 <?xml version="1.0"?>
 <robot xmlns:xacro="http://www.ros.org/wiki/xacro">
-  <xacro:macro name="arm_macro" params="id use_sim use_mock_hardware">
+  <xacro:macro name="arm_macro" params="id">
     <ros2_control name="arm_${id}" type="system">
       <xacro:unless value="$(arg use_mock_hardware)">

Commit message: Fix joint names, add velocity command interface

File: src/rai_description/urdf/rai.ros2_control.xacro (robot description, xacro)
@@ -20,11 +20,13 @@
         </xacro:unless>
       </xacro:if>
-      <joint name="$arm_revolute_${id}">
+      <joint name="arm_revolute_${id}">
         <command_interface name="position"/>
+        <command_interface name="velocity"/>
         <state_interface name="position"/>
         <state_interface name="velocity"/>
       </joint>
-      <joint name="$arm_slider_${id}">
+      <joint name="arm_slider_${id}">
         <command_interface name="position"/>
+        <command_interface name="velocity"/>
         <state_interface name="position"/>
         <state_interface name="velocity"/>
@@ -54,6 +56,7 @@
       </xacro:unless>
     </xacro:if>
-    <joint name="$canvas_revolute">
+    <joint name="canvas_revolute">
       <command_interface name="position"/>
+      <command_interface name="velocity"/>
       <state_interface name="position"/>
       <state_interface name="velocity"/>

Commit message: Initial implementation of ros2 control within simulation (#6)
* placeholder implementations

* implement package and cmakelists

* intermediate commit, before changing mock hardware params to args

* change params to args, add canvas

* move arm macros to control file

* remove params from arm macro

* add gazebo tag to urdf

* Update existing bringups to match sim/mock hardware patterns

* implement ros2_controllers

* Implement ros2 control launch file

* Add control to bringup

* fix ros2 control dependencies

* Fix fail fast bugs

* Fix joint names, add velocity command interface

* change duplicate joint controller to velocity

* Remove automatic joint state publisher start

* add rqt joint trajectory controller utility

* enable gazebo self collision checking

* Add joint trajectory gui task

File: src/rai_description/urdf/rai.ros2_control.xacro (robot description, xacro)
@@ -1,30 +1,32 @@
 <?xml version="1.0"?>
 <robot xmlns:xacro="http://www.ros.org/wiki/xacro">
-  <xacro:macro name="bot_ros2_control" params="name prefix use_mock_hardware">
-    <ros2_control name="${name}" type="system">
-      <!-- Physical hardware plugin-->
-      <xacro:unless value="${use_mock_hardware}">
+  <xacro:macro name="arm_macro" params="id">
+    <ros2_control name="arm_${id}" type="system">
+      <xacro:unless value="$(arg use_mock_hardware)">
         <hardware>
-          <plugin>odrive_ros2_control_plugin/ODriveHardwareInterface</plugin>
-          <param name="can">can0</param>
+          <plugin></plugin> #TODO Placeholder for real hardware
         </hardware>
       </xacro:unless>
-      <!-- Generic mock hardware motors-->
-      <!-- TODO Make it so that GazeboSimSystem is dependent on use_sim, and GenericSystem is dependent on !use_sim and use_mock_hardware-->
-      <xacro:if value="${use_mock_hardware}">
-        <hardware>
-          <plugin>gz_ros2_control/GazeboSimSystem</plugin>
-        </hardware>
+      <xacro:if value="$(arg use_mock_hardware)">
+        <xacro:if value="$(arg use_sim)">
+          <hardware>
+            <plugin>gz_ros2_control/GazeboSimSystem</plugin>
+          </hardware>
+        </xacro:if>
+        <xacro:unless value="$(arg use_sim)">
+          <hardware>
+            <plugin>mock_components/GenericSystem</plugin>
+          </hardware>
+        </xacro:unless>
       </xacro:if>
-      <!-- Odrive node ID setups-->
-      <joint name="${prefix}left_wheel_joint">
-        <param name="node_id">0</param>
-         <command_interface name="velocity"/>
+      <joint name="arm_revolute_${id}">
+        <command_interface name="position"/>
+        <command_interface name="velocity"/>
         <state_interface name="position"/>
         <state_interface name="velocity"/>
       </joint>
-      <joint name="${prefix}right_wheel_joint">
-        <param name="node_id">1</param>
-         <command_interface name="velocity"/>
+      <joint name="arm_slider_${id}">
+        <command_interface name="position"/>
+        <command_interface name="velocity"/>
         <state_interface name="position"/>
         <state_interface name="velocity"/>
@@ -32,3 +34,32 @@
     </ros2_control>
   </xacro:macro>
+  <xacro:arm_macro id ="1"/>
+  <xacro:arm_macro id ="2"/>
+  <xacro:arm_macro id ="3"/>
+  <xacro:arm_macro id ="4"/>
+  <ros2_control name="canvas" type="system">
+    <xacro:unless value="$(arg use_mock_hardware)">
+      <hardware>
+        <plugin></plugin> #TODO Placeholder for real hardware
+      </hardware>
+    </xacro:unless>
+    <xacro:if value="$(arg use_mock_hardware)">
+      <xacro:if value="$(arg use_sim)">
+        <hardware>
+          <plugin>gz_ros2_control/GazeboSimSystem</plugin>
+        </hardware>
+      </xacro:if>
+      <xacro:unless value="$(arg use_sim)">
+        <hardware>
+          <plugin>mock_components/GenericSystem</plugin>
+        </hardware>
+      </xacro:unless>
+    </xacro:if>
+    <joint name="canvas_revolute">
+      <command_interface name="position"/>
+      <command_interface name="velocity"/>
+      <state_interface name="position"/>
+      <state_interface name="velocity"/>
+    </joint>
+  </ros2_control>
 </robot>

File: src/rai_description/urdf/rai.urdf.xacro (robot description, xacro)
@@ -1,6 +1,9 @@
 <?xml version="1.0"?>
 <robot name="rai" xmlns:xacro="http://www.ros.org/wiki/xacro">
+    <xacro:arg name="use_sim" default="false"/>
+    <xacro:arg name="use_mock_hardware" default="false"/>
     <!-- Include generated urdf -->
     <xacro:include filename="$(find rai_description)/urdf/rai_geometry.urdf" />
+    <xacro:include filename="$(find rai_description)/urdf/rai.ros2_control.xacro" />
     <link name="world"/>
     <joint name="world_fixed" type="fixed">
@@ -8,3 +11,9 @@
         <child link="base_link"/>
     </joint>
+    <gazebo>
+        <self_collide>true</self_collide>
+        <plugin filename="gz_ros2_control-system" name="gz_ros2_control::GazeboSimROS2ControlPlugin">
+            <parameters>$(find rai_control)/config/ros2_controllers.yaml</parameters>
+        </plugin>
+    </gazebo>
 </robot>
