Commit message: Update URDF with pen frames

File: src/rai_description/urdf/rai_geometry.urdf (robot description, URDF)
Before this commit: robot robot, 11 links, 10 joints
Links:
- added link pen_1, mass 1e-9
- added link pen_2, mass 1e-9
- added link pen_3, mass 1e-9
- added link pen_4, mass 1e-9
Joints:
- added joint pen_1_frame: type fixed, parent arm, child pen_1, origin xyz=0.0002 0.0313875 -0.549649 rpy=-1.5708 0.821505 -0, axis 0 0 0
- added joint pen_2_frame: type fixed, parent arm_2, child pen_2, origin xyz=0.0002 0.0313875 -0.549649 rpy=-1.5708 0.821505 -0, axis 0 0 0
- added joint pen_3_frame: type fixed, parent arm_3, child pen_3, origin xyz=0.0002 0.0313875 -0.549649 rpy=-1.5708 0.821505 -0, axis 0 0 0
- added joint pen_4_frame: type fixed, parent arm_4, child pen_4, origin xyz=0.0002 0.0313875 -0.549649 rpy=-1.5708 0.821505 -0, axis 0 0 0
- joint arm_revolute_1: limit lower=-3.141592653589793 upper=3.141592653589793 effort=10 velocity=6 -> lower=-3.141592653589793 upper=3.141592653589793 effort=0.61 velocity=157
- joint arm_revolute_2: limit lower=-3.141592653589793 upper=3.141592653589793 effort=10 velocity=6 -> lower=-3.141592653589793 upper=3.141592653589793 effort=0.61 velocity=157
- joint arm_revolute_3: limit lower=-3.141592653589793 upper=3.141592653589793 effort=10 velocity=6 -> lower=-3.141592653589793 upper=3.141592653589793 effort=0.61 velocity=157
- joint arm_revolute_4: limit lower=-3.141592653589793 upper=3.141592653589793 effort=10 velocity=6 -> lower=-3.141592653589793 upper=3.141592653589793 effort=0.61 velocity=157
- joint arm_slider_1: limit lower=-0.277756 upper=0.0742877 effort=10 velocity=6 -> lower=-0.277756 upper=0.0742877 effort=90 velocity=0.25
- joint arm_slider_2: limit lower=-0.272538 upper=0.0795063 effort=10 velocity=6 -> lower=-0.272538 upper=0.0795063 effort=90 velocity=0.25
- joint arm_slider_3: limit lower=-0.228952 upper=0.123092 effort=10 velocity=6 -> lower=-0.228952 upper=0.123092 effort=90 velocity=0.25
- joint arm_slider_4: limit lower=-0.158753 upper=0.193291 effort=10 velocity=6 -> lower=-0.158753 upper=0.193291 effort=90 velocity=0.25
- joint canvas_revolute: limit effort=10 velocity=6 -> effort=1.45 velocity=157

Commit message: add dummy inertia to urdf

File: src/rai_description/urdf/rai_geometry.urdf (robot description, URDF)
Before this commit: robot rai, 15 links, 14 joints
Links:
- link base_link: mass 0 -> None
- link chassis: mass 0 -> 0.1

Commit message: Update arm homing positions

File: src/rai_description/urdf/rai_geometry.urdf (robot description, URDF)
Before this commit: robot rai, 15 links, 14 joints
Joints:
- joint arm_revolute_1: origin xyz=-0.306801 -0.306801 0.233705 rpy=-0 -0 1.41921 -> xyz=-0.306801 -0.306801 0.233705 rpy=-0 0 1.5708
- joint arm_revolute_2: origin xyz=0.306801 -0.306801 0.233705 rpy=-0 0 3.03808 -> xyz=0.306801 -0.306801 0.233705 rpy=0 0 -3.14159
- joint arm_revolute_3: origin xyz=0.306801 0.306801 0.233705 rpy=0 -0 -1.48206 -> xyz=0.306801 0.306801 0.233705 rpy=0 -0 -1.5708
- joint arm_revolute_4: origin xyz=-0.306801 0.306801 0.233705 rpy=-0 -0 -0.0856695 -> xyz=-0.306801 0.306801 0.233705 rpy=-0 -0 0
- joint arm_slider_1: limit lower=-0.277756 upper=0.0742877 effort=90 velocity=0.25 -> lower=-0.1778 upper=0.174244 effort=90 velocity=0.25; origin xyz=-0.260844 0.242656 -0.0135128 rpy=-1.5708 0 0.821505 -> xyz=-0.181234 0.181234 -0.0135128 rpy=-1.5708 0 0.785398
- joint arm_slider_2: limit lower=-0.272538 upper=0.0795063 effort=90 velocity=0.25 -> lower=-0.1778 upper=0.174244 effort=90 velocity=0.25; origin xyz=-0.257023 0.239102 -0.0135128 rpy=-1.5708 0 0.821505 -> xyz=-0.181234 0.181234 -0.0135128 rpy=-1.5708 0 0.785398
- joint arm_slider_3: limit lower=-0.228952 upper=0.123092 effort=90 velocity=0.25 -> lower=-0.1778 upper=0.174244 effort=90 velocity=0.25; origin xyz=-0.22511 0.209414 -0.0135128 rpy=-1.5708 0 0.821505 -> xyz=-0.181234 0.181234 -0.0135128 rpy=-1.5708 0 0.785398
- joint arm_slider_4: limit lower=-0.158753 upper=0.193291 effort=90 velocity=0.25 -> lower=-0.1778 upper=0.174244 effort=90 velocity=0.25; origin xyz=-0.173713 0.1616 -0.0135128 rpy=-1.5708 0 0.821505 -> xyz=-0.181234 0.181234 -0.0135128 rpy=-1.5708 0 0.785398
- joint canvas_revolute: origin xyz=-0 0 0.166624 rpy=-3.14159 0 -2.7447 -> xyz=-0 0 0.166624 rpy=3.14159 0 1.5708
